Commit message: Update champ.urdf

File: champ_description/urdf/champ.urdf (robot description, URDF)
Before this commit: robot champ, 29 links, 28 joints
Links:
- link base_link: geometry collision mesh filename=package://champ_description/meshes/chassis.stl scale=0.001 0.001 0.001; visual mesh filename=package://champ_description/meshes/chassis.stl scale=0.001 0.001 0.001
