Commit message: Update properties.urdf.xacro

File: champ_description/urdf/properties.urdf.xacro (robot description, xacro)
@@ -11,15 +11,15 @@
     <xacro:property name="hip_y_length" value="0.08" />
     <xacro:property name="hip_z_length" value="0.130" />
-    <xacro:property name="upper_leg_mesh_path" value="package://champ_description/meshes/upper_leg.stl" />
+    <xacro:property name="upper_leg_mesh_path" value="package://champ_description/meshes/femur.stl" />
     <xacro:property name="upper_leg_mass" value="0.125" />
     <xacro:property name="upper_leg_x_length" value="0.05" />
     <xacro:property name="upper_leg_y_length" value="0.03" />
     <xacro:property name="upper_leg_z_length" value="0.1905" />
-    <xacro:property name="lower_leg_mesh_path" value="package://champ_description/meshes/lower_leg.stl" />
+    <xacro:property name="lower_leg_mesh_path" value="package://champ_description/meshes/tibia.stl" />
     <xacro:property name="lower_leg_mass" value="0.125" />
     <xacro:property name="lower_leg_x_length" value="0.039" />
     <xacro:property name="lower_leg_y_length" value="0.022" />
     <xacro:property name="lower_leg_z_length" value="0.156" />
-    <xacro:property name="base_mesh_path" value="package://champ_description/meshes/base.stl" />
+    <xacro:property name="base_mesh_path" value="package://champ_description/meshes/chassis.stl" />
     <xacro:property name="base_mass" value="2.0" />
     <xacro:property name="base_x_length" value="0.5" />
