Commit message: Add files via upload

File: quadrubot_urdf_description/urdf/quadrubot_urdf.xacro (robot description, xacro)
@@ -24,5 +24,5 @@
   </collision>
 </link>
-<link name="LH_femur_1">
+<link name="LH_femur">
   <inertial>
     <origin xyz="0.007999966833522235 -0.00023763115376576605 -0.05206077683730421" rpy="0 0 0"/>
@@ -33,5 +33,5 @@
     <origin xyz="-0.08 -0.117973 -0.01085" rpy="0 0 0"/>
     <geometry>
-      <mesh filename="package://quadrubot_urdf_description/meshes/LH_femur_1.stl" scale="0.001 0.001 0.001"/>
+      <mesh filename="package://quadrubot_urdf_description/meshes/femur.stl" scale="0.001 0.001 0.001"/>
     </geometry>
     <material name="silver"/>
@@ -40,9 +40,9 @@
     <origin xyz="-0.08 -0.117973 -0.01085" rpy="0 0 0"/>
     <geometry>
-      <mesh filename="package://quadrubot_urdf_description/meshes/LH_femur_1.stl" scale="0.001 0.001 0.001"/>
-    </geometry>
-  </collision>
-</link>
-<link name="hip_right_v6_1">
+      <mesh filename="package://quadrubot_urdf_description/meshes/femur.stl" scale="0.001 0.001 0.001"/>
+    </geometry>
+  </collision>
+</link>
+<link name="LH_hip">
   <inertial>
     <origin xyz="-0.004396117471655678 -0.0280002447595447 -0.010174881105460217" rpy="0 0 0"/>
@@ -53,5 +53,5 @@
     <origin xyz="0.05025 0.079973 -0.01085" rpy="0 0 0"/>
     <geometry>
-      <mesh filename="package://quadrubot_urdf_description/meshes/hip_right_v6_1.stl" scale="0.001 0.001 0.001"/>
+      <mesh filename="package://quadrubot_urdf_description/meshes/L_hip.stl" scale="0.001 0.001 0.001"/>
     </geometry>
     <material name="silver"/>
@@ -60,9 +60,9 @@
     <origin xyz="0.05025 0.079973 -0.01085" rpy="0 0 0"/>
     <geometry>
-      <mesh filename="package://quadrubot_urdf_description/meshes/hip_right_v6_1.stl" scale="0.001 0.001 0.001"/>
-    </geometry>
-  </collision>
-</link>
-<link name="hip_left_v2__1__1">
+      <mesh filename="package://quadrubot_urdf_description/meshes/L_hip.stl" scale="0.001 0.001 0.001"/>
+    </geometry>
+  </collision>
+</link>
+<link name="RH_hip">
   <inertial>
     <origin xyz="0.004396117471655747 -0.02800024475954467 -0.01017488110546024" rpy="0 0 0"/>
@@ -73,5 +73,5 @@
     <origin xyz="-0.05025 0.079973 -0.01085" rpy="0 0 0"/>
     <geometry>
-      <mesh filename="package://quadrubot_urdf_description/meshes/hip_left_v2__1__1.stl" scale="0.001 0.001 0.001"/>
+      <mesh filename="package://quadrubot_urdf_description/meshes/R_hip.stl" scale="0.001 0.001 0.001"/>
     </geometry>
     <material name="silver"/>
@@ -80,9 +80,9 @@
     <origin xyz="-0.05025 0.079973 -0.01085" rpy="0 0 0"/>
     <geometry>
-      <mesh filename="package://quadrubot_urdf_description/meshes/hip_left_v2__1__1.stl" scale="0.001 0.001 0.001"/>
-    </geometry>
-  </collision>
-</link>
-<link name="hip_left_v2_1">
+      <mesh filename="package://quadrubot_urdf_description/meshes/R_hip.stl" scale="0.001 0.001 0.001"/>
+    </geometry>
+  </collision>
+</link>
+<link name="RF_hip">
   <inertial>
     <origin xyz="0.004396117471655685 0.028000244759544643 -0.010174881105460238" rpy="0 0 0"/>
@@ -93,5 +93,5 @@
     <origin xyz="-0.05025 -0.079973 -0.01085" rpy="0 0 0"/>
     <geometry>
-      <mesh filename="package://quadrubot_urdf_description/meshes/hip_left_v2_1.stl" scale="0.001 0.001 0.001"/>
+      <mesh filename="package://quadrubot_urdf_description/meshes/R_hip.stl" scale="0.001 0.001 0.001"/>
     </geometry>
     <material name="silver"/>
@@ -100,18 +100,18 @@
     <origin xyz="-0.05025 -0.079973 -0.01085" rpy="0 0 0"/>
     <geometry>
-      <mesh filename="package://quadrubot_urdf_description/meshes/hip_left_v2_1.stl" scale="0.001 0.001 0.001"/>
-    </geometry>
-  </collision>
-</link>
-<link name="hip_right_v6__1__1">
-  <inertial>
-    <origin xyz="-0.0023806840931287626 0.028000244759544643 -0.010825272803639804" rpy="0 0 0"/>
+      <mesh filename="package://quadrubot_urdf_description/meshes/R_hip.stl" scale="0.001 0.001 0.001"/>
+    </geometry>
+  </collision>
+</link>
+<link name="LF_hip">
+  <inertial>
+    <origin xyz="-0.0043961174716557055 0.02800024475954467 -0.010174881105460226" rpy="0 0 0"/>
     <mass value="0.7107341380350983"/>
-    <inertia ixx="0.00028" iyy="0.000197" izz="0.000287" ixy="0.0" iyz="-0.0" ixz="-1e-06"/>
+    <inertia ixx="0.00028" iyy="0.000197" izz="0.000287" ixy="0.0" iyz="-0.0" ixz="1e-06"/>
   </inertial>
   <visual>
     <origin xyz="0.05025 -0.079973 -0.01085" rpy="0 0 0"/>
     <geometry>
-      <mesh filename="package://quadrubot_urdf_description/meshes/hip_right_v6__1__1.stl" scale="0.001 0.001 0.001"/>
+      <mesh filename="package://quadrubot_urdf_description/meshes/L_hip.stl" scale="0.001 0.001 0.001"/>
     </geometry>
     <material name="silver"/>
@@ -120,9 +120,9 @@
     <origin xyz="0.05025 -0.079973 -0.01085" rpy="0 0 0"/>
     <geometry>
-      <mesh filename="package://quadrubot_urdf_description/meshes/hip_right_v6__1__1.stl" scale="0.001 0.001 0.001"/>
-    </geometry>
-  </collision>
-</link>
-<link name="LF_femur_1">
+      <mesh filename="package://quadrubot_urdf_description/meshes/L_hip.stl" scale="0.001 0.001 0.001"/>
+    </geometry>
+  </collision>
+</link>
+<link name="LF_femur">
   <inertial>
     <origin xyz="0.00799996683352211 -2.4475954325808846e-07 -0.052061320285349356" rpy="0 0 0"/>
@@ -133,5 +133,5 @@
     <origin xyz="-0.08 0.097973 -0.01085" rpy="0 0 0"/>
     <geometry>
-      <mesh filename="package://quadrubot_urdf_description/meshes/LF_femur_1.stl" scale="0.001 0.001 0.001"/>
+      <mesh filename="package://quadrubot_urdf_description/meshes/femur.stl" scale="0.001 0.001 0.001"/>
     </geometry>
     <material name="silver"/>
@@ -140,9 +140,9 @@
     <origin xyz="-0.08 0.097973 -0.01085" rpy="0 0 0"/>
     <geometry>
-      <mesh filename="package://quadrubot_urdf_description/meshes/LF_femur_1.stl" scale="0.001 0.001 0.001"/>
-    </geometry>
-  </collision>
-</link>
-<link name="LF_foot_1">
+      <mesh filename="package://quadrubot_urdf_description/meshes/femur.stl" scale="0.001 0.001 0.001"/>
+    </geometry>
+  </collision>
+</link>
+<link name="LF_foot">
   <inertial>
     <origin xyz="3.0443070174607234e-06 0.00011974192622413171 -0.0036898240176088948" rpy="0 0 0"/>
@@ -153,5 +153,5 @@
     <origin xyz="-0.08675 0.189835 0.193867" rpy="0 0 0"/>
     <geometry>
-      <mesh filename="package://quadrubot_urdf_description/meshes/LF_foot_1.stl" scale="0.001 0.001 0.001"/>
+      <mesh filename="package://quadrubot_urdf_description/meshes/foot.stl" scale="0.001 0.001 0.001"/>
     </geometry>
     <material name="silver"/>
@@ -160,9 +160,9 @@
     <origin xyz="-0.08675 0.189835 0.193867" rpy="0 0 0"/>
     <geometry>
-      <mesh filename="package://quadrubot_urdf_description/meshes/LF_foot_1.stl" scale="0.001 0.001 0.001"/>
-    </geometry>
-  </collision>
-</link>
-<link name="LH_tibia_1">
+      <mesh filename="package://quadrubot_urdf_description/meshes/foot.stl" scale="0.001 0.001 0.001"/>
+    </geometry>
+  </collision>
+</link>
+<link name="LH_tibia">
   <inertial>
     <origin xyz="-0.009622915734244925 -0.04376557953636863 -0.04018872915444033" rpy="0 0 0"/>
@@ -173,5 +173,5 @@
     <origin xyz="-0.096 -0.117425 0.109149" rpy="0 0 0"/>
     <geometry>
-      <mesh filename="package://quadrubot_urdf_description/meshes/LH_tibia_1.stl" scale="0.001 0.001 0.001"/>
+      <mesh filename="package://quadrubot_urdf_description/meshes/L_tibia.stl" scale="0.001 0.001 0.001"/>
     </geometry>
     <material name="silver"/>
@@ -180,9 +180,9 @@
     <origin xyz="-0.096 -0.117425 0.109149" rpy="0 0 0"/>
     <geometry>
-      <mesh filename="package://quadrubot_urdf_description/meshes/LH_tibia_1.stl" scale="0.001 0.001 0.001"/>
-    </geometry>
-  </collision>
-</link>
-<link name="LH_foot_1">
+      <mesh filename="package://quadrubot_urdf_description/meshes/L_tibia.stl" scale="0.001 0.001 0.001"/>
+    </geometry>
+  </collision>
+</link>
+<link name="LH_foot">
   <inertial>
     <origin xyz="3.0443070160174335e-06 0.0001029473381414861 -0.0036904656393174917" rpy="0 0 0"/>
@@ -193,5 +193,5 @@
     <origin xyz="-0.08675 -0.025177 0.193445" rpy="0 0 0"/>
     <geometry>
-      <mesh filename="package://quadrubot_urdf_description/meshes/LH_foot_1.stl" scale="0.001 0.001 0.001"/>
+      <mesh filename="package://quadrubot_urdf_description/meshes/foot.stl" scale="0.001 0.001 0.001"/>
     </geometry>
     <material name="silver"/>
@@ -200,69 +200,69 @@
     <origin xyz="-0.08675 -0.025177 0.193445" rpy="0 0 0"/>
     <geometry>
-      <mesh filename="package://quadrubot_urdf_description/meshes/LH_foot_1.stl" scale="0.001 0.001 0.001"/>
-    </geometry>
-  </collision>
-</link>
-<link name="RH_femur_1">
-  <inertial>
-    <origin xyz="0.000603951922637222 0.027070665878713845 -0.04517997413000263" rpy="0 0 0"/>
+      <mesh filename="package://quadrubot_urdf_description/meshes/foot.stl" scale="0.001 0.001 0.001"/>
+    </geometry>
+  </collision>
+</link>
+<link name="RH_femur">
+  <inertial>
+    <origin xyz="-0.007999966833522998 0.05206156504489351 -1.528291382335567e-15" rpy="0 0 0"/>
     <mass value="0.3755220822299566"/>
-    <inertia ixx="0.000591" iyy="0.000442" izz="0.000194" ixy="-4.9e-05" iyz="0.000251" ixz="8e-05"/>
-  </inertial>
-  <visual>
-    <origin xyz="0.079457 -0.117973 -0.005192" rpy="0 0 0"/>
-    <geometry>
-      <mesh filename="package://quadrubot_urdf_description/meshes/RH_femur_1.stl" scale="0.001 0.001 0.001"/>
-    </geometry>
-    <material name="silver"/>
-  </visual>
-  <collision>
-    <origin xyz="0.079457 -0.117973 -0.005192" rpy="0 0 0"/>
-    <geometry>
-      <mesh filename="package://quadrubot_urdf_description/meshes/RH_femur_1.stl" scale="0.001 0.001 0.001"/>
-    </geometry>
-  </collision>
-</link>
-<link name="RH_tibia_1">
-  <inertial>
-    <origin xyz="0.020747841120931143 0.0006404282430508834 -0.05650079826905842" rpy="0 0 0"/>
+    <inertia ixx="0.000606" iyy="2.3e-05" izz="0.000598" ixy="0.0" iyz="0.0" ixz="0.0"/>
+  </inertial>
+  <visual>
+    <origin xyz="0.08 -0.117973 -0.01085" rpy="0 0 0"/>
+    <geometry>
+      <mesh filename="package://quadrubot_urdf_description/meshes/femur.stl" scale="0.001 0.001 0.001"/>
+    </geometry>
+    <material name="silver"/>
+  </visual>
+  <collision>
+    <origin xyz="0.08 -0.117973 -0.01085" rpy="0 0 0"/>
+    <geometry>
+      <mesh filename="package://quadrubot_urdf_description/meshes/femur.stl" scale="0.001 0.001 0.001"/>
+    </geometry>
+  </collision>
+</link>
+<link name="RH_tibia">
+  <inertial>
+    <origin xyz="0.009622915728666817 -0.04358118970385538 -0.040388529207220226" rpy="0 0 0"/>
     <mass value="0.31452387445863506"/>
-    <inertia ixx="0.000582" iyy="0.000587" izz="5.4e-05" ixy="1.5e-05" iyz="-7.8e-05" ixz="9.9e-05"/>
-  </inertial>
-  <visual>
-    <origin xyz="0.07567 -0.18037 0.098482" rpy="0 0 0"/>
-    <geometry>
-      <mesh filename="package://quadrubot_urdf_description/meshes/RH_tibia_1.stl" scale="0.001 0.001 0.001"/>
-    </geometry>
-    <material name="silver"/>
-  </visual>
-  <collision>
-    <origin xyz="0.07567 -0.18037 0.098482" rpy="0 0 0"/>
-    <geometry>
-      <mesh filename="package://quadrubot_urdf_description/meshes/RH_tibia_1.stl" scale="0.001 0.001 0.001"/>
-    </geometry>
-  </collision>
-</link>
-<link name="RH_foot_1">
-  <inertial>
-    <origin xyz="0.00045810214696603846 0.002813546931035832 -0.002345860838545988" rpy="0 0 0"/>
+    <inertia ixx="0.0006" iyy="0.000206" izz="0.000417" ixy="-5e-06" iyz="-0.000266" ixz="-4e-06"/>
+  </inertial>
+  <visual>
+    <origin xyz="0.096 -0.237973 -0.01085" rpy="0 0 0"/>
+    <geometry>
+      <mesh filename="package://quadrubot_urdf_description/meshes/R_tibia.stl" scale="0.001 0.001 0.001"/>
+    </geometry>
+    <material name="silver"/>
+  </visual>
+  <collision>
+    <origin xyz="0.096 -0.237973 -0.01085" rpy="0 0 0"/>
+    <geometry>
+      <mesh filename="package://quadrubot_urdf_description/meshes/R_tibia.stl" scale="0.001 0.001 0.001"/>
+    </geometry>
+  </collision>
+</link>
+<link name="RH_foot">
+  <inertial>
+    <origin xyz="3.1106399750457925e-06 0.00011923144531283958 -0.0036898240176075625" rpy="0 0 0"/>
     <mass value="0.010948791496213523"/>
-    <inertia ixx="1e-06" iyy="1e-06" izz="1e-06" ixy="0.0" iyz="-0.0" ixz="0.0"/>
-  </inertial>
-  <visual>
-    <origin xyz="0.042823 -0.181413 0.2194" rpy="0 0 0"/>
-    <geometry>
-      <mesh filename="package://quadrubot_urdf_description/meshes/RH_foot_1.stl" scale="0.001 0.001 0.001"/>
-    </geometry>
-    <material name="silver"/>
-  </visual>
-  <collision>
-    <origin xyz="0.042823 -0.181413 0.2194" rpy="0 0 0"/>
-    <geometry>
-      <mesh filename="package://quadrubot_urdf_description/meshes/RH_foot_1.stl" scale="0.001 0.001 0.001"/>
-    </geometry>
-  </collision>
-</link>
-<link name="RF_femur_1">
+    <inertia ixx="1e-06" iyy="1e-06" izz="2e-06" ixy="-0.0" iyz="0.0" ixz="0.0"/>
+  </inertial>
+  <visual>
+    <origin xyz="0.08675 -0.146112 0.073867" rpy="0 0 0"/>
+    <geometry>
+      <mesh filename="package://quadrubot_urdf_description/meshes/foot.stl" scale="0.001 0.001 0.001"/>
+    </geometry>
+    <material name="silver"/>
+  </visual>
+  <collision>
+    <origin xyz="0.08675 -0.146112 0.073867" rpy="0 0 0"/>
+    <geometry>
+      <mesh filename="package://quadrubot_urdf_description/meshes/foot.stl" scale="0.001 0.001 0.001"/>
+    </geometry>
+  </collision>
+</link>
+<link name="RF_femur">
   <inertial>
     <origin xyz="-0.007999966833521999 -2.447595432442107e-07 -0.05206132028534933" rpy="0 0 0"/>
@@ -273,5 +273,5 @@
     <origin xyz="0.08 0.097973 -0.01085" rpy="0 0 0"/>
     <geometry>
-      <mesh filename="package://quadrubot_urdf_description/meshes/RF_femur_1.stl" scale="0.001 0.001 0.001"/>
+      <mesh filename="package://quadrubot_urdf_description/meshes/femur.stl" scale="0.001 0.001 0.001"/>
     </geometry>
     <material name="silver"/>
@@ -280,9 +280,9 @@
     <origin xyz="0.08 0.097973 -0.01085" rpy="0 0 0"/>
     <geometry>
-      <mesh filename="package://quadrubot_urdf_description/meshes/RF_femur_1.stl" scale="0.001 0.001 0.001"/>
-    </geometry>
-  </collision>
-</link>
-<link name="RF_tibia_1">
+      <mesh filename="package://quadrubot_urdf_description/meshes/femur.stl" scale="0.001 0.001 0.001"/>
+    </geometry>
+  </collision>
+</link>
+<link name="RF_tibia">
   <inertial>
     <origin xyz="0.009622915728667969 -0.0435816792229442 -0.040388529207220275" rpy="0 0 0"/>
@@ -293,5 +293,5 @@
     <origin xyz="0.096 0.097973 0.10915" rpy="0 0 0"/>
     <geometry>
-      <mesh filename="package://quadrubot_urdf_description/meshes/RF_tibia_1.stl" scale="0.001 0.001 0.001"/>
+      <mesh filename="package://quadrubot_urdf_description/meshes/R_tibia.stl" scale="0.001 0.001 0.001"/>
     </geometry>
     <material name="silver"/>
@@ -300,9 +300,9 @@
     <origin xyz="0.096 0.097973 0.10915" rpy="0 0 0"/>
     <geometry>
-      <mesh filename="package://quadrubot_urdf_description/meshes/RF_tibia_1.stl" scale="0.001 0.001 0.001"/>
-    </geometry>
-  </collision>
-</link>
-<link name="RF_foot_1">
+      <mesh filename="package://quadrubot_urdf_description/meshes/R_tibia.stl" scale="0.001 0.001 0.001"/>
+    </geometry>
+  </collision>
+</link>
+<link name="RF_foot">
   <inertial>
     <origin xyz="3.1106399753649816e-06 0.00011974192622413171 -0.0036898240176076458" rpy="0 0 0"/>
@@ -313,5 +313,5 @@
     <origin xyz="0.08675 0.189835 0.193867" rpy="0 0 0"/>
     <geometry>
-      <mesh filename="package://quadrubot_urdf_description/meshes/RF_foot_1.stl" scale="0.001 0.001 0.001"/>
+      <mesh filename="package://quadrubot_urdf_description/meshes/foot.stl" scale="0.001 0.001 0.001"/>
     </geometry>
     <material name="silver"/>
@@ -320,9 +320,9 @@
     <origin xyz="0.08675 0.189835 0.193867" rpy="0 0 0"/>
     <geometry>
-      <mesh filename="package://quadrubot_urdf_description/meshes/RF_foot_1.stl" scale="0.001 0.001 0.001"/>
-    </geometry>
-  </collision>
-</link>
-<link name="LF_tibia_1">
+      <mesh filename="package://quadrubot_urdf_description/meshes/foot.stl" scale="0.001 0.001 0.001"/>
+    </geometry>
+  </collision>
+</link>
+<link name="LF_tibia">
   <inertial>
     <origin xyz="-0.009622915734244203 -0.043581684927930076 -0.040388533468682014" rpy="0 0 0"/>
@@ -333,5 +333,5 @@
     <origin xyz="-0.096 0.097973 0.10915" rpy="0 0 0"/>
     <geometry>
-      <mesh filename="package://quadrubot_urdf_description/meshes/LF_tibia_1.stl" scale="0.001 0.001 0.001"/>
+      <mesh filename="package://quadrubot_urdf_description/meshes/L_tibia.stl" scale="0.001 0.001 0.001"/>
     </geometry>
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